File: docs/projects/993-programmable-rear-panel/electronics/kicad/coupon-e0.kicad_sch (KiCad schematic)
At the start: 18 parts, among them J1 3V3 LAB, J2 LOGIC / DK USB SEPARE, U7 SN74LVC125APW, U8 SN74LVC1G04DBVR

Commit message: docs(993-rear-panel): translate CSV data and KiCad schematic text to English
Finishes the English pass started in PR 146. Free-text columns of bom.csv,
measurements.csv, coupon-bom.csv and coupon-wiring.csv, plus the titles,
notes, sheet name and two component values of the three KiCad sheets, are now
English. Identifiers, nets, pins, references, numeric values, statuses and CSV
columns are unchanged; the schematic test expects the two new values.

The review PDF is re-exported with kicad/kicad:9.0.2 (network disabled):
schematic test OK, ERC 0 errors 0 warnings, pages reviewed visually. The
verification page records the run and the export's environment dependence.

Co-Authored-By: Claude Opus 5.5 <noreply@anthropic.com>
Parts:
- J2: value LOGIC / DK USB SEPARE -> LOGIC / DK USB SEPARATE
- S1: value COUPURE LED -> LED CUTOFF
Other:
- sheet Matrice LED 16 x 8 renamed LED matrix 16 x 8
- note added: "C7 near U7; C8 near U8. Values and sequences to measure on the bench."
- note added: "COUPON E0 / 16 x 8 red LEDs / 3.3 V on the bench"
- note added: "Current-limited lab power supply. Sources off before wiring."
- note added: "DISPLAY_EN low -> BLANK high -> black. MCU stuck high: use S1."
- note added: "NOT VALIDATED FOR MANUFACTURING - no connection to the vehicle"
- note added: "No DK VDD/VBUS on J1/J2. DK GPIO pins to be defined."
- note added: "S1 cuts the LED rail; C10 discharges through R15. No hardware watchdog."
- note added: "Sheets linked by global labels. KiCad 9.0.2 symbols; no footprint assigned."
- note removed: "Alimentation de laboratoire limitee en courant. Sources coupees avant cablage."
- note removed: "Aucun VDD/VBUS du DK sur J1/J2. Broches GPIO DK a definir."
- note removed: "C7 pres U7; C8 pres U8. Valeurs et sequences a mesurer au banc."
- note removed: "COUPON E0 / 16 x 8 LED rouges / 3,3 V au banc"
- note removed: "DISPLAY_EN bas -> BLANK haut -> noir. MCU bloque haut : utiliser S1."
- note removed: "Liaisons entre feuilles par labels globaux. Symboles KiCad 9.0.2; aucune empreinte attribuee."
- note removed: "NON VALIDE POUR FABRICATION - pas de raccordement au vehicule"
- note removed: "S1 coupe le rail LED; C10 se decharge par R15. Pas de watchdog materiel."
- title: Coupon E0 - Alimentation et commande -> Coupon E0 - Power and control
Changed lines of the file:
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@@
-(kicad_sch (version 20250114) (generator "eeschema") (paper "A3") (title_block (title "Coupon E0 - Alimentation et commande") (date "2026-10-02") (rev "E0.1") (comment 1 "NON VALIDE POUR FABRICATION - BANC 3.3 V UNIQUEMENT") (comment 2 "Empreintes non attribuees; aucun PCB ni validation physique"))
-(text "COUPON E0 / 16 x 8 LED rouges / 3,3 V au banc" (at 15.24 15.24 0) (effects (font (size 2.5 2.5)) (justify left top)))
-(text "NON VALIDE POUR FABRICATION - pas de raccordement au vehicule" (at 15.24 21.59 0) (effects (font (size 1.5 1.5)) (justify left top)))
-(text "Alimentation de laboratoire limitee en courant. Sources coupees avant cablage." (at 15.24 27.94 0) (effects (font (size 1.5 1.5)) (justify left top)))
+(kicad_sch (version 20250114) (generator "eeschema") (paper "A3") (title_block (title "Coupon E0 - Power and control") (date "2026-10-02") (rev "E0.1") (comment 1 "NOT VALIDATED FOR MANUFACTURING - 3.3 V BENCH ONLY") (comment 2 "Footprints not assigned; no PCB and no physical validation"))
+(text "COUPON E0 / 16 x 8 red LEDs / 3.3 V on the bench" (at 15.24 15.24 0) (effects (font (size 2.5 2.5)) (justify left top)))
+(text "NOT VALIDATED FOR MANUFACTURING - no connection to the vehicle" (at 15.24 21.59 0) (effects (font (size 1.5 1.5)) (justify left top)))
+(text "Current-limited lab power supply. Sources off before wiring." (at 15.24 27.94 0) (effects (font (size 1.5 1.5)) (justify left top)))
 (symbol (lib_id "Connector_Generic:Conn_01x02") (at 50.8 50.8 0) (unit 1) (in_bom yes) (on_board yes) (dnp no) (property "Reference" "J1" (at 54.8 49.3 0) (effects (font (size 1.0 1.0)) (justify left))) (property "Value" "3V3 LAB" (at 54.8 52.3 0) (effects (font (size 1.0 1.0)) (justify left))) (property "Footprint" "" (at 54.8 52.3 0) (effects (font (size 1.0 1.0)) (justify left) (hide yes))) (property "Datasheet" "~" (at 54.8 52.3 0) (effects (font (size 1.0 1.0)) (justify left) (hide yes))) (pin "1") (pin "2") (instances (project "coupon-e0" (path "/1851a418-39cb-5a7b-850e-cab555b60ad9" (reference "J1") (unit 1)))))
 (wire (pts (xy 45.72 50.8) (xy 40.64 50.8)) (stroke (width 0) (type default)))
@@
 (wire (pts (xy 45.72 53.34) (xy 40.64 53.34)) (stroke (width 0) (type default)))
 (global_label "GND" (shape passive) (at 40.64 53.34 180) (effects (font (size 0.95 0.95)) (justify right)) (property "Intersheetrefs" "${INTERSHEET_REFS}" (at 40.64 53.34 0) (effects (font (size 1.0 1.0)) (hide yes))))
-(symbol (lib_id "Switch:SW_SPST") (at 114.3 50.8 0) (unit 1) (in_bom yes) (on_board yes) (dnp no) (property "Reference" "S1" (at 118.3 49.3 0) (effects (font (size 1.0 1.0)) (justify left))) (property "Value" "COUPURE LED" (at 118.3 52.3 0) (effects (font (size 1.0 1.0)) (justify left))) (property "Footprint" "" (at 118.3 52.3 0) (effects (font (size 1.0 1.0)) (justify left) (hide yes))) (property "Datasheet" "~" (at 118.3 52.3 0) (effects (font (size 1.0 1.0)) (justify left) (hide yes))) (pin "1") (pin "2") (instances (project "coupon-e0" (path "/1851a418-39cb-5a7b-850e-cab555b60ad9" (reference "S1") (unit 1)))))
+(symbol (lib_id "Switch:SW_SPST") (at 114.3 50.8 0) (unit 1) (in_bom yes) (on_board yes) (dnp no) (property "Reference" "S1" (at 118.3 49.3 0) (effects (font (size 1.0 1.0)) (justify left))) (property "Value" "LED CUTOFF" (at 118.3 52.3 0) (effects (font (size 1.0 1.0)) (justify left))) (property "Footprint" "" (at 118.3 52.3 0) (effects (font (size 1.0 1.0)) (justify left) (hide yes))) (property "Datasheet" "~" (at 118.3 52.3 0) (effects (font (size 1.0 1.0)) (justify left) (hide yes))) (pin "1") (pin "2") (instances (project "coupon-e0" (path "/1851a418-39cb-5a7b-850e-cab555b60ad9" (reference "S1") (unit 1)))))
 (wire (pts (xy 109.22 50.8) (xy 104.14 50.8)) (stroke (width 0) (type default)))
 (global_label "VCC_3V3" (shape passive) (at 104.14 50.8 180) (effects (font (size 0.95 0.95)) (justify right)) (property "Intersheetrefs" "${INTERSHEET_REFS}" (at 104.14 50.8 0) (effects (font (size 1.0 1.0)) (hide yes))))
@@
 (wire (pts (xy 281.94 60.96) (xy 281.94 66.04)) (stroke (width 0) (type default)))
 (global_label "GND" (shape passive) (at 281.94 66.04 0) (effects (font (size 0.95 0.95)) (justify left)) (property "Intersheetrefs" "${INTERSHEET_REFS}" (at 281.94 66.04 0) (effects (font (size 1.0 1.0)) (hide yes))))
-(text "S1 coupe le rail LED; C10 se decharge par R15. Pas de watchdog materiel." (at 106.68 83.82 0) (effects (font (size 1.5 1.5)) (justify left top)))
-(symbol (lib_id "Connector_Generic:Conn_01x06") (at 55.88 114.3 0) (unit 1) (in_bom yes) (on_board yes) (dnp no) (property "Reference" "J2" (at 59.88 112.8 0) (effects (font (size 1.0 1.0)) (justify left))) (property "Value" "LOGIC / DK USB SEPARE" (at 59.88 115.8 0) (effects (font (size 1.0 1.0)) (justify left))) (property "Footprint" "" (at 59.88 115.8 0) (effects (font (size 1.0 1.0)) (justify left) (hide yes))) (property "Datasheet" "~" (at 59.88 115.8 0) (effects (font (size 1.0 1.0)) (justify left) (hide yes))) (pin "1") (pin "2") (pin "3") (pin "4") (pin "5") (pin "6") (instances (project "coupon-e0" (path "/1851a418-39cb-5a7b-850e-cab555b60ad9" (reference "J2") (unit 1)))))
+(text "S1 cuts the LED rail; C10 discharges through R15. No hardware watchdog." (at 106.68 83.82 0) (effects (font (size 1.5 1.5)) (justify left top)))
+(symbol (lib_id "Connector_Generic:Conn_01x06") (at 55.88 114.3 0) (unit 1) (in_bom yes) (on_board yes) (dnp no) (property "Reference" "J2" (at 59.88 112.8 0) (effects (font (size 1.0 1.0)) (justify left))) (property "Value" "LOGIC / DK USB SEPARATE" (at 59.88 115.8 0) (effects (font (size 1.0 1.0)) (justify left))) (property "Footprint" "" (at 59.88 115.8 0) (effects (font (size 1.0 1.0)) (justify left) (hide yes))) (property "Datasheet" "~" (at 59.88 115.8 0) (effects (font (size 1.0 1.0)) (justify left) (hide yes))) (pin "1") (pin "2") (pin "3") (pin "4") (pin "5") (pin "6") (instances (project "coupon-e0" (path "/1851a418-39cb-5a7b-850e-cab555b60ad9" (reference "J2") (unit 1)))))
 (wire (pts (xy 50.8 109.22) (xy 45.72 109.22)) (stroke (width 0) (type default)))
 (global_label "GND" (shape passive) (at 45.72 109.22 180) (effects (font (size 0.95 0.95)) (justify right)) (property "Intersheetrefs" "${INTERSHEET_REFS}" (at 45.72 109.22 0) (effects (font (size 1.0 1.0)) (hide yes))))
@@
 (wire (pts (xy 50.8 121.92) (xy 45.72 121.92)) (stroke (width 0) (type default)))
 (global_label "GND" (shape passive) (at 45.72 121.92 180) (effects (font (size 0.95 0.95)) (justify right)) (property "Intersheetrefs" "${INTERSHEET_REFS}" (at 45.72 121.92 0) (effects (font (size 1.0 1.0)) (hide yes))))
-(text "Aucun VDD/VBUS du DK sur J1/J2. Broches GPIO DK a definir." (at 15.24 139.7 0) (effects (font (size 1.5 1.5)) (justify left top)))
+(text "No DK VDD/VBUS on J1/J2. DK GPIO pins to be defined." (at 15.24 139.7 0) (effects (font (size 1.5 1.5)) (justify left top)))
 (symbol (lib_id "rear_panel_e0:SN74LVC125APW") (at 139.7 109.22 0) (unit 1) (in_bom yes) (on_board yes) (dnp no) (property "Reference" "U7" (at 139.7 103.22 0) (effects (font (size 1.0 1.0)))) (property "Value" "SN74LVC125APW" (at 139.7 100.22 0) (effects (font (size 1.0 1.0)) (hide yes))) (property "Footprint" "" (at 139.7 100.22 0) (effects (font (size 1.0 1.0)) (hide yes))) (property "Datasheet" "http://www.ti.com/lit/gpn/sn74LVC125" (at 139.7 100.22 0) (effects (font (size 1.0 1.0)) (hide yes))) (pin "2") (pin "1") (pin "3") (instances (project "coupon-e0" (path "/1851a418-39cb-5a7b-850e-cab555b60ad9" (reference "U7") (unit 1)))))
 (wire (pts (xy 132.08 109.22) (xy 127 109.22)) (stroke (width 0) (type default)))
@@
 (wire (pts (xy 368.3 210.82) (xy 368.3 215.9)) (stroke (width 0) (type default)))
 (global_label "GND" (shape passive) (at 368.3 215.9 0) (effects (font (size 0.95 0.95)) (justify left)) (property "Intersheetrefs" "${INTERSHEET_REFS}" (at 368.3 215.9 0) (effects (font (size 1.0 1.0)) (hide yes))))
-(text "DISPLAY_EN bas -> BLANK haut -> noir. MCU bloque haut : utiliser S1." (at 15.24 234.95 0) (effects (font (size 1.5 1.5)) (justify left top)))
-(text "C7 pres U7; C8 pres U8. Valeurs et sequences a mesurer au banc." (at 15.24 241.3 0) (effects (font (size 1.5 1.5)) (justify left top)))
+(text "DISPLAY_EN low -> BLANK high -> black. MCU stuck high: use S1." (at 15.24 234.95 0) (effects (font (size 1.5 1.5)) (justify left top)))
+(text "C7 near U7; C8 near U8. Values and sequences to measure on the bench." (at 15.24 241.3 0) (effects (font (size 1.5 1.5)) (justify left top)))
 (sheet (at 25.4 254) (size 65 25) (stroke (width .15) (type default)) (fill (color 0 0 0 0)) (property "Sheetname" "Six drivers TLC5947DAP" (at 57.9 252 0) (effects (font (size 1.0 1.0))))(property "Sheetfile" "drivers.kicad_sch" (at 57.9 282 0) (effects (font (size 1.0 1.0)))) (instances (project "coupon-e0" (path "/1851a418-39cb-5a7b-850e-cab555b60ad9" (page "2")))))
-(sheet (at 124.46 254) (size 65 25) (stroke (width .15) (type default)) (fill (color 0 0 0 0)) (property "Sheetname" "Matrice LED 16 x 8" (at 156.96 252 0) (effects (font (size 1.0 1.0))))(property "Sheetfile" "leds.kicad_sch" (at 156.96 282 0) (effects (font (size 1.0 1.0)))) (instances (project "coupon-e0" (path "/1851a418-39cb-5a7b-850e-cab555b60ad9" (page "3")))))
-(text "Liaisons entre feuilles par labels globaux.\nSymboles KiCad 9.0.2; aucune empreinte attribuee." (at 220.98 248.92 0) (effects (font (size 1.1 1.1)) (justify left top)))
+(sheet (at 124.46 254) (size 65 25) (stroke (width .15) (type default)) (fill (color 0 0 0 0)) (property "Sheetname" "LED matrix 16 x 8" (at 156.96 252 0) (effects (font (size 1.0 1.0))))(property "Sheetfile" "leds.kicad_sch" (at 156.96 282 0) (effects (font (size 1.0 1.0)))) (instances (project "coupon-e0" (path "/1851a418-39cb-5a7b-850e-cab555b60ad9" (page "3")))))
+(text "Sheets linked by global labels.\nKiCad 9.0.2 symbols; no footprint assigned." (at 220.98 248.92 0) (effects (font (size 1.1 1.1)) (justify left top)))
 (sheet_instances (path "/" (page "1")))
 )
