File: docs/projects/993-programmable-rear-panel/electronics/kicad/drivers.kicad_sch (KiCad schematic)
At the start: 26 parts, among them U1 TLC5947DAP, U2 TLC5947DAP, U3 TLC5947DAP, U4 TLC5947DAP, U5 TLC5947DAP, U6 TLC5947DAP

Commit message: docs(993-rear-panel): translate CSV data and KiCad schematic text to English
Finishes the English pass started in PR 146. Free-text columns of bom.csv,
measurements.csv, coupon-bom.csv and coupon-wiring.csv, plus the titles,
notes, sheet name and two component values of the three KiCad sheets, are now
English. Identifiers, nets, pins, references, numeric values, statuses and CSV
columns are unchanged; the schematic test expects the two new values.

The review PDF is re-exported with kicad/kicad:9.0.2 (network disabled):
schematic test OK, ERC 0 errors 0 warnings, pages reviewed visually. The
verification page records the run and the export's environment dependence.

Co-Authored-By: Claude Opus 5.5 <noreply@anthropic.com>
Other:
- note added: "6 x TLC5947DAP / static outputs / chain SIN -> U1 -> ... -> U6"
- note added: "DAP only. Thermal pad = KiCad pin 33, to connect to GND. IREF: 20k 1% / driver."
- note added: "U6 OUT8..23 not connected; PWM data = 0. C1..C6 as close as possible to driver VCC."
- note removed: "6 x TLC5947DAP / sorties statiques / chaine SIN -> U1 -> ... -> U6"
- note removed: "DAP uniquement. Pad thermique = broche KiCad 33, a relier a GND. IREF : 20k 1% / driver."
- note removed: "U6 OUT8..23 non connectees; donnees PWM = 0. C1..C6 au plus pres des VCC des drivers."
- title: Coupon E0 - Drivers et points de test -> Coupon E0 - Drivers and test points
Changed lines of the file:
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@@
-(kicad_sch (version 20250114) (generator "eeschema") (paper "A3") (title_block (title "Coupon E0 - Drivers et points de test") (date "2026-10-02") (rev "E0.1") (comment 1 "NON VALIDE POUR FABRICATION - BANC 3.3 V UNIQUEMENT") (comment 2 "Empreintes non attribuees; aucun PCB ni validation physique"))
-(text "6 x TLC5947DAP / sorties statiques / chaine SIN -> U1 -> ... -> U6" (at 15.24 15.24 0) (effects (font (size 2 2)) (justify left top)))
-(text "DAP uniquement. Pad thermique = broche KiCad 33, a relier a GND. IREF : 20k 1% / driver." (at 15.24 22.86 0) (effects (font (size 1.3 1.3)) (justify left top)))
+(kicad_sch (version 20250114) (generator "eeschema") (paper "A3") (title_block (title "Coupon E0 - Drivers and test points") (date "2026-10-02") (rev "E0.1") (comment 1 "NOT VALIDATED FOR MANUFACTURING - 3.3 V BENCH ONLY") (comment 2 "Footprints not assigned; no PCB and no physical validation"))
+(text "6 x TLC5947DAP / static outputs / chain SIN -> U1 -> ... -> U6" (at 15.24 15.24 0) (effects (font (size 2 2)) (justify left top)))
+(text "DAP only. Thermal pad = KiCad pin 33, to connect to GND. IREF: 20k 1% / driver." (at 15.24 22.86 0) (effects (font (size 1.3 1.3)) (justify left top)))
 (symbol (lib_id "Driver_LED:TLC5947DAP") (at 76.2 83.82 0) (unit 1) (in_bom yes) (on_board yes) (dnp no) (property "Reference" "U1" (at 62.23 45.72 0) (effects (font (size 1.0 1.0)))) (property "Value" "TLC5947DAP" (at 62.23 48.26 0) (effects (font (size 1.0 1.0)))) (property "Footprint" "" (at 62.23 43.18 0) (effects (font (size 1.0 1.0)) (hide yes))) (property "Datasheet" "http://www.ti.com/lit/ds/symlink/tlc5947.pdf" (at 76.2 83.82 0) (effects (font (size 1.0 1.0)) (hide yes))) (pin "31") (pin "2") (pin "30") (pin "3") (pin "4") (pin "29") (pin "1") (pin "33") (pin "32") (pin "5") (pin "6") (pin "7") (pin "8") (pin "9") (pin "10") (pin "11") (pin "12") (pin "13") (pin "14") (pin "15") (pin "16") (pin "17") (pin "18") (pin "19") (pin "20") (pin "21") (pin "22") (pin "23") (pin "24") (pin "25") (pin "26") (pin "27") (pin "28") (instances (project "coupon-e0" (path "/1851a418-39cb-5a7b-850e-cab555b60ad9/d65a47c0-f40b-54eb-9822-b2e6360cf081" (reference "U1") (unit 1)))))
 (wire (pts (xy 73.66 119.38) (xy 73.66 124.46)) (stroke (width 0) (type default)))
@@
 (wire (pts (xy 203.2 265.43) (xy 203.2 270.51)) (stroke (width 0) (type default)))
 (global_label "SOUT_TEST" (shape passive) (at 203.2 270.51 0) (effects (font (size 0.95 0.95)) (justify left)) (property "Intersheetrefs" "${INTERSHEET_REFS}" (at 203.2 270.51 0) (effects (font (size 1.0 1.0)) (hide yes))))
-(text "U6 OUT8..23 non connectees; donnees PWM = 0. C1..C6 au plus pres des VCC des drivers." (at 15.24 248.92 0) (effects (font (size 1.1 1.1)) (justify left top)))
+(text "U6 OUT8..23 not connected; PWM data = 0. C1..C6 as close as possible to driver VCC." (at 15.24 248.92 0) (effects (font (size 1.1 1.1)) (justify left top)))
 )
