File: docs/projects/993-programmable-rear-panel/electronics/kicad/leds.kicad_sch (KiCad schematic)
At the start: 128 parts

Commit message: docs(993-rear-panel): translate CSV data and KiCad schematic text to English
Finishes the English pass started in PR 146. Free-text columns of bom.csv,
measurements.csv, coupon-bom.csv and coupon-wiring.csv, plus the titles,
notes, sheet name and two component values of the three KiCad sheets, are now
English. Identifiers, nets, pins, references, numeric values, statuses and CSV
columns are unchanged; the schematic test expects the two new values.

The review PDF is re-exported with kicad/kicad:9.0.2 (network disabled):
schematic test OK, ERC 0 errors 0 warnings, pages reviewed visually. The
verification page records the run and the export's environment dependence.

Co-Authored-By: Claude Opus 5.5 <noreply@anthropic.com>
Other:
- note added: "1 x 0.5 mm package != pitch. Compare 2.5 / 4 mm on the bench. Footprint and polarity to review before routing."
- note added: "D1..D128: APHHS1005LSECK/J3-PF / anode (2) on VLED_3V3"
- note added: "Logical view of the LED face: rows left to right. Schematic not to scale, no PCB placement."
- note added: "One output per cathode. The 16 remaining U6 outputs are not connected. All footprints remain to be defined."
- note removed: "Boitier 1 x 0,5 mm != pas. Comparer 2,5 / 4 mm au banc. Empreinte et polarite a revoir avant routage."
- note removed: "D1..D128 : APHHS1005LSECK/J3-PF / anode (2) sur VLED_3V3"
- note removed: "Une sortie par cathode. Les 16 sorties restantes de U6 sont non connectees. Toutes les empreintes restent a definir."
- note removed: "Vue logique face LED : lignes de gauche a droite. Schema sans echelle ni placement PCB."
- title: Coupon E0 - Matrice rouge 16 x 8 -> Coupon E0 - Red matrix 16 x 8
Changed lines of the file:
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@@
-(kicad_sch (version 20250114) (generator "eeschema") (paper "A3") (title_block (title "Coupon E0 - Matrice rouge 16 x 8") (date "2026-10-02") (rev "E0.1") (comment 1 "NON VALIDE POUR FABRICATION - BANC 3.3 V UNIQUEMENT") (comment 2 "Empreintes non attribuees; aucun PCB ni validation physique"))
-(text "D1..D128 : APHHS1005LSECK/J3-PF / anode (2) sur VLED_3V3" (at 15.24 15.24 0) (effects (font (size 2 2)) (justify left top)))
-(text "Vue logique face LED : lignes de gauche a droite. Schema sans echelle ni placement PCB." (at 15.24 22.86 0) (effects (font (size 1.3 1.3)) (justify left top)))
-(text "Boitier 1 x 0,5 mm != pas. Comparer 2,5 / 4 mm au banc. Empreinte et polarite a revoir avant routage." (at 15.24 29.21 0) (effects (font (size 1.3 1.3)) (justify left top)))
+(kicad_sch (version 20250114) (generator "eeschema") (paper "A3") (title_block (title "Coupon E0 - Red matrix 16 x 8") (date "2026-10-02") (rev "E0.1") (comment 1 "NOT VALIDATED FOR MANUFACTURING - 3.3 V BENCH ONLY") (comment 2 "Footprints not assigned; no PCB and no physical validation"))
+(text "D1..D128: APHHS1005LSECK/J3-PF / anode (2) on VLED_3V3" (at 15.24 15.24 0) (effects (font (size 2 2)) (justify left top)))
+(text "Logical view of the LED face: rows left to right. Schematic not to scale, no PCB placement." (at 15.24 22.86 0) (effects (font (size 1.3 1.3)) (justify left top)))
+(text "1 x 0.5 mm package != pitch. Compare 2.5 / 4 mm on the bench. Footprint and polarity to review before routing." (at 15.24 29.21 0) (effects (font (size 1.3 1.3)) (justify left top)))
 (global_label "VLED_3V3" (shape passive) (at 22.86 44.45 180) (effects (font (size 0.95 0.95)) (justify right)) (property "Intersheetrefs" "${INTERSHEET_REFS}" (at 22.86 44.45 0) (effects (font (size 1.0 1.0)) (hide yes))))
 (symbol (lib_id "Device:LED") (at 35.56 52.07 90) (unit 1) (in_bom yes) (on_board yes) (dnp no) (property "Reference" "D1" (at 40.56 50.57 90) (effects (font (size 1.0 1.0)) (justify left))) (property "Value" "APHHS1005LSECK/J3-PF" (at 40.56 53.57 90) (effects (font (size 1.0 1.0)) (justify left) (hide yes))) (property "Footprint" "" (at 40.56 53.57 90) (effects (font (size 1.0 1.0)) (justify left) (hide yes))) (property "Datasheet" "~" (at 40.56 53.57 90) (effects (font (size 1.0 1.0)) (justify left) (hide yes))) (pin "1") (pin "2") (instances (project "coupon-e0" (path "/1851a418-39cb-5a7b-850e-cab555b60ad9/edd98504-fd32-5273-9127-bc95e1137841" (reference "D1") (unit 1)))))
@@
 (wire (pts (xy 378.46 242.57) (xy 378.46 245.11)) (stroke (width 0) (type default)))
 (global_label "LED_K128" (shape passive) (at 378.46 245.11 0) (effects (font (size 0.95 0.95)) (justify left)) (property "Intersheetrefs" "${INTERSHEET_REFS}" (at 378.46 245.11 0) (effects (font (size 1.0 1.0)) (hide yes))))
-(text "Une sortie par cathode. Les 16 sorties restantes de U6 sont non connectees. Toutes les empreintes restent a definir." (at 15.24 262.89 0) (effects (font (size 1.1 1.1)) (justify left top)))
+(text "One output per cathode. The 16 remaining U6 outputs are not connected. All footprints remain to be defined." (at 15.24 262.89 0) (effects (font (size 1.1 1.1)) (justify left top)))
 )
